File: Protoboard_power_supply.sch (KiCad schematic (older format))
At the start: 16 parts, among them CON1 BARREL_JACK, P1 USB_A, P2 OUT2, P3 OUT1, P4 SELECTOR, SW1 SW_DPDT_x2, U1 LM1117-3.3, U2 LM1117-5.0

Commit message: Placa terminada
Parts:
- removed P1: USB_A, symbol conn:USB_A
- removed SW1: SW_DPDT_x2, symbol switches:SW_DPDT_x2
- added P1: USB_OTG, Connectors:USB_Mini-B, symbol conn:USB_OTG
- added SW1: SW_DPDT_x2, Buttons_Switches_THT:SW_CuK_JS202011CQN_DPDT_Straight, symbol Switch:SW_DPDT_x2
- C1, C2: footprint (none) -> Capacitors_SMD:C_0805_HandSoldering
- C3: footprint (none) -> Capacitors_THT:CP_Radial_D4.0mm_P1.50mm
- C4: footprint (none) -> Capacitors_THT:CP_Radial_D6.3mm_P2.50mm
- CON1: footprint (none) -> Connectors:JACK_ALIM
- D1: footprint Diodes_THT:D_DO-41_SOD81_Horizontal_RM10 -> Diodes_SMD:D_SMA
- D2: footprint (none) -> LEDs:LED_0805_HandSoldering
- F1: footprint (none) -> Fuse_Holders_and_Fuses:Fuse_SMD1206_Reflow
- P2, P3, P4: footprint (none) -> Pin_Headers:Pin_Header_Straight_2x03_Pitch2.54mm
- R1: footprint (none) -> Resistors_SMD:R_0805_HandSoldering
- U1, U2: footprint (none) -> TO_SOT_Packages_SMD:SOT-223
Connections:
- net 5V: now also SW1.6 (C)
- net GND: now also P1.5 (GND), P1.6 (shield)
- net VBUS: now also P1.1 (VBUS)
- net at CON1.1: now also SW1.2 (B)
- net at D1.2 (A): now also SW1.3 (C)
- net at F1.1: now also SW1.5 (B)
- no-connect marks 4 -> 5
Changed lines of the file:
@@
 F 0 "CON1" H 3481 3575 50  0000 C CNN
 F 1 "BARREL_JACK" H 3481 3484 50  0000 C CNN
-F 2 "" H 3500 3250 50  0001 C CNN
+F 2 "Connectors:JACK_ALIM" H 3500 3250 50  0001 C CNN
 F 3 "" H 3500 3250 50  0001 C CNN
 	1    3500 3250
 	1    0    0    -1
-$EndComp
-$Comp
-L conn:USB_A P1
-U 1 1 5C0CF730
-P 3050 4250
-F 0 "P1" V 3123 4438 50  0000 L CNN
-F 1 "USB_A" V 3032 4438 50  0000 L CNN
-F 2 "" V 3000 4150 50  0001 C CNN
-F 3 "" V 3000 4150 50  0001 C CNN
-	1    3050 4250
-	0    -1   1    0
 $EndComp
 $Comp
@@
 F 0 "U1" H 8000 3492 50  0000 C CNN
 F 1 "LM1117-3.3" H 8000 3401 50  0000 C CNN
-F 2 "" H 8000 3250 50  0001 C CNN
+F 2 "TO_SOT_Packages_SMD:SOT-223" H 8000 3250 50  0001 C CNN
 F 3 "http://www.ti.com/lit/ds/symlink/lm1117.pdf" H 8000 3250 50  0001 C CNN
 	1    8000 3250
@@
 F 0 "U2" H 6150 3492 50  0000 C CNN
 F 1 "LM1117-5.0" H 6150 3401 50  0000 C CNN
-F 2 "" H 6150 3250 50  0001 C CNN
+F 2 "TO_SOT_Packages_SMD:SOT-223" H 6150 3250 50  0001 C CNN
 F 3 "http://www.ti.com/lit/ds/symlink/lm1117.pdf" H 6150 3250 50  0001 C CNN
 	1    6150 3250
@@
 F 0 "D2" H 5150 4785 50  0000 C CNN
 F 1 "Power" H 5150 4694 50  0000 C CNN
-F 2 "" V 5150 4550 50  0001 C CNN
+F 2 "LEDs:LED_0805_HandSoldering" V 5150 4550 50  0001 C CNN
 F 3 "~" V 5150 4550 50  0001 C CNN
 	1    5150 4550
@@
 F 0 "D1" H 5100 3466 50  0000 C CNN
 F 1 "1N4001" H 5100 3375 50  0000 C CNN
-F 2 "Diodes_THT:D_DO-41_SOD81_Horizontal_RM10" H 5100 3075 50  0001 C CNN
+F 2 "Diodes_SMD:D_SMA" H 5100 3075 50  0001 C CNN
 F 3 "http://www.vishay.com/docs/88503/1n4001.pdf" H 5100 3250 50  0001 C CNN
 	1    5100 3250
@@
 F 0 "R1" H 5209 4296 50  0000 L CNN
 F 1 "470R" H 5209 4205 50  0000 L CNN
-F 2 "" H 5150 4250 50  0001 C CNN
+F 2 "Resistors_SMD:R_0805_HandSoldering" H 5150 4250 50  0001 C CNN
 F 3 "" H 5150 4250 50  0001 C CNN
 	1    5150 4250
@@
 F 0 "C3" H 8588 3446 50  0000 L CNN
 F 1 "10uF" H 8588 3355 50  0000 L CNN
-F 2 "" H 8500 3400 50  0001 C CNN
+F 2 "Capacitors_THT:CP_Radial_D4.0mm_P1.50mm" H 8500 3400 50  0001 C CNN
 F 3 "" H 8500 3400 50  0001 C CNN
 	1    8500 3400
@@
 F 0 "C4" H 6738 3446 50  0000 L CNN
 F 1 "100uF" H 6738 3355 50  0000 L CNN
-F 2 "" H 6650 3400 50  0001 C CNN
+F 2 "Capacitors_THT:CP_Radial_D6.3mm_P2.50mm" H 6650 3400 50  0001 C CNN
 F 3 "" H 6650 3400 50  0001 C CNN
 	1    6650 3400
@@
 L CH340G_D-SUN-V3.0-cache:GND #PWR01
 U 1 1 5C0DBCF6
-P 2950 4600
-F 0 "#PWR01" H 2950 4350 50  0001 C CNN
-F 1 "GND" H 2955 4427 50  0000 C CNN
-F 2 "" H 2950 4600 60  0000 C CNN
-F 3 "" H 2950 4600 60  0000 C CNN
-	1    2950 4600
-	1    0    0    -1
-$EndComp
-Wire Wire Line
-	2950 4550 2950 4600
+P 2900 4700
+F 0 "#PWR01" H 2900 4450 50  0001 C CNN
+F 1 "GND" H 2905 4527 50  0000 C CNN
+F 2 "" H 2900 4700 60  0000 C CNN
+F 3 "" H 2900 4700 60  0000 C CNN
+	1    2900 4700
+	1    0    0    -1
+$EndComp
 $Comp
 L CH340G_D-SUN-V3.0-cache:GND #PWR02
@@
 	1    0    0    -1
 $EndComp
-Wire Wire Line
-	3450 4600 3450 4350
-Wire Wire Line
-	3450 4350 3350 4350
-NoConn ~ 3350 4150
-NoConn ~ 3350 4250
 Connection ~ 7500 3250
 Wire Wire Line
@@
 	7050 3250 7500 3250
 $Comp
-L switches:SW_DPDT_x2 SW1
-U 1 1 5C0E2AD9
-P 4250 3150
-F 0 "SW1" H 4250 3435 50  0000 C CNN
-F 1 "SW_DPDT_x2" H 4250 3344 50  0000 C CNN
-F 2 "" H 4250 3150 50  0001 C CNN
-F 3 "" H 4250 3150 50  0001 C CNN
-	1    4250 3150
-	1    0    0    -1
-$EndComp
-$Comp
-L switches:SW_DPDT_x2 SW1
-U 2 1 5C0E2B64
-P 4250 4050
-F 0 "SW1" H 4250 4335 50  0000 C CNN
-F 1 "SW_DPDT_x2" H 4250 4244 50  0000 C CNN
-F 2 "" H 4250 4050 50  0001 C CNN
-F 3 "" H 4250 4050 50  0001 C CNN
-	2    4250 4050
-	1    0    0    -1
-$EndComp
-$Comp
 L power:VBUS #PWR03
 U 1 1 5C0DD51C
@@
 	1    0    0    -1
 $EndComp
-Wire Wire Line
-	3350 4050 3500 4050
 Wire Wire Line
 	3500 4050 3500 4000
@@
 F 0 "F1" V 3695 4050 50  0000 C CNN
 F 1 "500mA" V 3786 4050 50  0000 C CNN
-F 2 "" H 3950 3850 50  0001 L CNN
+F 2 "Fuse_Holders_and_Fuses:Fuse_SMD1206_Reflow" H 3950 3850 50  0001 L CNN
 F 3 "" H 3900 4050 50  0001 C CNN
 	1    3900 4050
@@
 F 0 "P2" H 6300 4765 50  0000 C CNN
 F 1 "OUT2" H 6300 4674 50  0000 C CNN
-F 2 "" H 6300 3250 50  0001 C CNN
+F 2 "Pin_Headers:Pin_Header_Straight_2x03_Pitch2.54mm" H 6300 3250 50  0001 C CNN
 F 3 "" H 6300 3250 50  0001 C CNN
 	1    6300 4450
@@
 F 0 "P3" H 7300 4765 50  0000 C CNN
 F 1 "OUT1" H 7300 4674 50  0000 C CNN
-F 2 "" H 7300 3250 50  0001 C CNN
+F 2 "Pin_Headers:Pin_Header_Straight_2x03_Pitch2.54mm" H 7300 3250 50  0001 C CNN
 F 3 "" H 7300 3250 50  0001 C CNN
 	1    7300 4450
@@
 F 0 "P4" H 8450 4815 50  0000 C CNN
 F 1 "SELECTOR" H 8450 4724 50  0000 C CNN
-F 2 "" H 8450 3300 50  0001 C CNN
+F 2 "Pin_Headers:Pin_Header_Straight_2x03_Pitch2.54mm" H 8450 3300 50  0001 C CNN
 F 3 "" H 8450 3300 50  0001 C CNN
 	1    8450 4500
@@
 F 0 "C1" H 5559 3446 50  0000 R CNN
 F 1 "100nF" H 5559 3355 50  0000 R CNN
-F 2 "" H 5650 3400 50  0001 C CNN
+F 2 "Capacitors_SMD:C_0805_HandSoldering" H 5650 3400 50  0001 C CNN
 F 3 "" H 5650 3400 50  0001 C CNN
 	1    5650 3400
@@
 F 0 "C2" H 7409 3446 50  0000 R CNN
 F 1 "100nF" H 7409 3355 50  0000 R CNN
-F 2 "" H 7500 3400 50  0001 C CNN
+F 2 "Capacitors_SMD:C_0805_HandSoldering" H 7500 3400 50  0001 C CNN
 F 3 "" H 7500 3400 50  0001 C CNN
 	1    7500 3400
 	1    0    0    -1
 $EndComp
+$Comp
+L Switch:SW_DPDT_x2 SW1
+U 1 1 5C0D853B
+P 4250 3150
+F 0 "SW1" H 4250 3435 50  0000 C CNN
+F 1 "SW_DPDT_x2" H 4250 3344 50  0000 C CNN
+F 2 "Buttons_Switches_THT:SW_CuK_JS202011CQN_DPDT_Straight" H 4250 3150 50  0001 C CNN
+F 3 "" H 4250 3150 50  0001 C CNN
+	1    4250 3150
+	1    0    0    -1
+$EndComp
+$Comp
+L Switch:SW_DPDT_x2 SW1
+U 2 1 5C0D85D8
+P 4250 4050
+F 0 "SW1" H 4250 4335 50  0000 C CNN
+F 1 "SW_DPDT_x2" H 4250 4244 50  0000 C CNN
+F 2 "Buttons_Switches_THT:SW_CuK_JS202011CQN_DPDT_Straight" H 4250 4050 50  0001 C CNN
+F 3 "" H 4250 4050 50  0001 C CNN
+	2    4250 4050
+	1    0    0    -1
+$EndComp
+$Comp
+L conn:USB_OTG P1
+U 1 1 5C0DA9AE
+P 3000 4250
+F 0 "P1" V 2575 4174 50  0000 C CNN
+F 1 "USB_OTG" V 2666 4174 50  0000 C CNN
+F 2 "Connectors:USB_Mini-B" V 2950 4150 50  0001 C CNN
+F 3 "" V 2950 4150 50  0001 C CNN
+	1    3000 4250
+	0    -1   1    0
+$EndComp
+Wire Wire Line
+	3300 4450 3450 4450
+Wire Wire Line
+	3450 4450 3450 4600
+Wire Wire Line
+	3300 4050 3500 4050
+NoConn ~ 3300 4150
+NoConn ~ 3300 4250
+NoConn ~ 3300 4350
+Wire Wire Line
+	2900 4650 2900 4700
 $EndSCHEMATC
