File: Protoboard_power_supply.kicad_pcb (KiCad board)
At the start: 2 copper layers, 50 x 27.9 mm, 17 parts, among them CON1 BARREL_JACK, P1 USB_OTG, P2 OUT2, P3 OUT1, P4 SELECTOR, SW1 SW_DPDT_x2, U1 LM1117-3.3, U2 LM1117-5.0

Commit message: Mandado a fabrica
Parts:
- added ?: , Aesthetics:OSHW-LOGO-S, F.Cu at (157.2, 88.6)
Other:
- board text added: "OFF"
- board text added: "ON"
Changed lines of the file:
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@@
   (general
     (thickness 1.6)
-    (drawings 20)
+    (drawings 22)
     (tracks 109)
     (zones 0)
-    (modules 17)
+    (modules 18)
     (nets 17)
   )
@@
     (visible_elements FFFFFF7F)
     (pcbplotparams
-      (layerselection 0x3ffff_80000001)
-      (usegerberextensions true)
+      (layerselection 0x110f0_ffffffff)
+      (usegerberextensions false)
       (usegerberattributes true)
       (usegerberadvancedattributes false)
       (creategerberjobfile false)
-      (excludeedgelayer true)
+      (excludeedgelayer false)
       (linewidth 0.127000)
       (plotframeref false)
       (viasonmask false)
       (mode 1)
-      (useauxorigin false)
+      (useauxorigin true)
       (hpglpennumber 1)
       (hpglpenspeed 20)
@@
       (psa4output false)
       (plotreference true)
-      (plotvalue true)
+      (plotvalue false)
       (plotinvisibletext false)
       (padsonsilk false)
@@
     (tags "Fuse Sicherung SMD1206 Littlefuse-Wickmann Reflow ")
     (attr smd)
-    (fp_text reference F1 (at -0.1 -2.75 270) (layer F.SilkS)
+    (fp_text reference F1 (at -3.048 0) (layer F.SilkS)
       (effects (font (size 1 1) (thickness 0.15)))
     )
@@
       (xy -2.2225 3.559306) (xy -2.2225 2.921)) (layer B.SilkS) (width 0.01))
   )
+  (module Aesthetics:OSHW-LOGO-S (layer F.Cu)
+    (at 157.226 88.646)
+    (descr "OPEN-SOURCE HARDWARE (OSHW) LOGO - SMALL - SILKSCREEN")
+    (tags "OPEN-SOURCE HARDWARE (OSHW) LOGO - SMALL - SILKSCREEN")
+    (attr virtual)
+    (fp_text reference "" (at 0 0) (layer F.SilkS)
+      (effects (font (size 1.524 1.524) (thickness 0.15)))
+    )
+    (fp_text value "" (at 0 0) (layer F.SilkS)
+      (effects (font (size 1.524 1.524) (thickness 0.15)))
+    )
+    (fp_poly (pts (xy 0.3937 0.9525) (xy 0.5461 0.87376) (xy 0.92202 1.1811) (xy 1.1811 0.92202)
+      (xy 0.87376 0.5461) (xy 0.9525 0.3937) (xy 1.0033 0.23114) (xy 1.48844 0.18034)
+      (xy 1.48844 -0.18034) (xy 1.0033 -0.23114) (xy 0.9525 -0.3937) (xy 0.87376 -0.5461)
+      (xy 1.1811 -0.92202) (xy 0.92202 -1.1811) (xy 0.5461 -0.87376) (xy 0.3937 -0.9525)
+      (xy 0.23114 -1.0033) (xy 0.18034 -1.48844) (xy -0.18034 -1.48844) (xy -0.23114 -1.0033)
+      (xy -0.3937 -0.9525) (xy -0.5461 -0.87376) (xy -0.92202 -1.1811) (xy -1.1811 -0.92202)
+      (xy -0.87376 -0.5461) (xy -0.9525 -0.3937) (xy -1.0033 -0.23114) (xy -1.48844 -0.18034)
+      (xy -1.48844 0.18034) (xy -1.0033 0.23114) (xy -0.9525 0.3937) (xy -0.87376 0.5461)
+      (xy -1.1811 0.92202) (xy -0.92202 1.1811) (xy -0.5461 0.87376) (xy -0.3937 0.9525)
+      (xy -0.1778 0.4318) (xy -0.27432 0.37846) (xy -0.3556 0.30226) (xy -0.41656 0.21082)
+      (xy -0.45466 0.10922) (xy -0.46736 0) (xy -0.45466 -0.10922) (xy -0.41402 -0.2159)
+      (xy -0.35052 -0.30734) (xy -0.2667 -0.38354) (xy -0.16764 -0.43434) (xy -0.06096 -0.46228)
+      (xy 0.0508 -0.46482) (xy 0.16002 -0.43942) (xy 0.25908 -0.38862) (xy 0.34544 -0.31496)
+      (xy 0.40894 -0.22352) (xy 0.45212 -0.11938) (xy 0.46736 -0.01016) (xy 0.4572 0.09906)
+      (xy 0.4191 0.20574) (xy 0.35814 0.29972) (xy 0.27686 0.37592) (xy 0.1778 0.4318)) (layer F.SilkS) (width 0.01))
+  )
+  (gr_text OFF (at 144.018 97.79) (layer F.SilkS)
+    (effects (font (size 0.8 0.8) (thickness 0.127)))
+  )
+  (gr_text ON (at 150.114 104.648) (layer F.SilkS)
+    (effects (font (size 0.8 0.8) (thickness 0.127)))
+  )
   (gr_text "Protoboard Power Supply\nV1.0" (at 168.656 88.392) (layer B.SilkS)
